File: KiCad/ExICE-M.sch (KiCad schematic (older format))
At the start: 71 parts, among them J1 PSS-710103-07, M1 MK06-4.5, M2 MK06-4.5, Q1 PT26-21C/TR8, Q2 PT26-21C/TR8, Q3 PT26-21C/TR8, Q4 PT26-21C/TR8, SW1 CUS-12TB, U1 MR25H40CDF, U10 MA700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

Commit message: KiCadバージョンアップ
Parts:
- BT1, M1, M2: symbol Conn_01x02 -> ExICE-M-rescue:Conn_01x02
- C1, C10, C11, C13, C14, C15, C16, C17, C18, C2, C3, C4, C5, C6, C7, C8, C9: symbol C_Small -> ExICE-M-rescue:C_Small
- D1, LD1, LD10, LD11, LD12, LD2, LD3, LD4, LD5, LD6, LD7, LD8, LD9: symbol LED -> ExICE-M-rescue:LED
- D2: symbol D_Schottky -> ExICE-M-rescue:D_Schottky
- J1: symbol Conn_01x07 -> ExICE-M-rescue:Conn_01x07
- L1: symbol L -> ExICE-M-rescue:L
- PAD1, PAD2, PAD3, PAD4: symbol Conn_01x04 -> ExICE-M-rescue:Conn_01x04
- Q1, Q2, Q3, Q4: symbol Q_Photo_NPN -> ExICE-M-rescue:Q_Photo_NPN
- R1, R10, R11, R12, R13, R14, R15, R16, R2, R3, R4, R5, R6, R7, R8, R9: symbol R -> ExICE-M-rescue:R
- SW1: symbol SW_Push_SPDT -> ExICE-M-rescue:SW_Push_SPDT
- U1: symbol MR25H40CDF -> ExICE-M:MR25H40CDF
- U10, U9: symbol MA700 -> ExICE-M:MA700
- U2: symbol NCV8705MT30TCG -> ExICE-M:NCV8705MT30TCG
- U3: symbol LTC4054ES5-4.2 -> ExICE-M:LTC4054ES5-4.2
- U4: symbol DRV8836 -> ExICE-M:DRV8836
- U5: symbol MIC2291-15YML -> ExICE-M:MIC2291-15YML
- U6: symbol STM32F411CEUx -> ExICE-M:STM32F411CEUx
- U7: symbol MAX7375AXR805+T -> ExICE-M:MAX7375AXR805+T
- U8: symbol ICM-20648 -> ExICE-M:ICM-20648
